File: board/afd/afd.kicad_pcb (KiCad board)
At the start: 2 copper layers, 0 parts

Commit message: Checkpoint.
Parts:
- added C1: 10 uF, Capacitor_SMD:C_1206_3216Metric_Pad1.33x1.80mm_HandSolder, F.Cu at (94.0, 116.8)
- added C2: 0.1 uF 20V ceramic, Capacitor_SMD:C_1206_3216Metric_Pad1.33x1.80mm_HandSolder, F.Cu at (125.7, 68.6)
- added C3: 22 uF, Capacitor_SMD:C_1206_3216Metric_Pad1.33x1.80mm_HandSolder, F.Cu at (106.0, 116.8)
- added C4: 0.1 uF 20V ceramic, Capacitor_SMD:C_1206_3216Metric_Pad1.33x1.80mm_HandSolder, F.Cu at (100.0, 116.8)
- added D1: Z0103MN, Package_TO_SOT_SMD:SOT-223, F.Cu at (106.7, 126.0)
- added D2: Z0103MN, Package_TO_SOT_SMD:SOT-223, F.Cu at (222.8, 59.4)
- added D3: Z0103MN, Package_TO_SOT_SMD:SOT-223, F.Cu at (132.4, 126.0)
- added D4: Z0103MN, Package_TO_SOT_SMD:SOT-223, F.Cu at (222.8, 75.2)
- added D5: Z0103MN, Package_TO_SOT_SMD:SOT-223, F.Cu at (158.2, 126.0)
- added D6: Z0103MN, Package_TO_SOT_SMD:SOT-223, F.Cu at (222.8, 91.0)
- added D7: Z0103MN, Package_TO_SOT_SMD:SOT-223, F.Cu at (183.9, 126.0)
- added D8: Z0103MN, Package_TO_SOT_SMD:SOT-223, F.Cu at (222.8, 106.8)
- added DS1: IEL-O-VI_C63.396.208-02, jdn_library:C63.396.208-02, F.Cu at (113.1, 85.2)
- added J1: ICSP Connector, Connector_PinHeader_2.54mm:PinHeader_1x05_P2.54mm_Vertical, F.Cu at (100.3, 58.4)
- added J2: GPIO Connector, Connector_PinHeader_2.54mm:PinHeader_1x05_P2.54mm_Vertical, F.Cu at (120.7, 58.4)
- added J3: Input Connector, Connector_PinHeader_2.54mm:PinHeader_1x06_P2.54mm_Vertical, F.Cu at (92.7, 82.5)
- added J4: Output Connector, Connector_PinHeader_2.54mm:PinHeader_1x06_P2.54mm_Vertical, F.Cu at (132.1, 82.5)
- added L1: 2.2 uH, Inductor_SMD:L_2816_7142Metric_Pad3.20x4.45mm_HandSolder, F.Cu at (128.3, 63.5)
- added R1: 10 Kohm, Resistor_SMD:R_1206_3216Metric_Pad1.30x1.75mm_HandSolder, F.Cu at (131.1, 74.9)
- added R10: 390, Resistor_SMD:R_1206_3216Metric_Pad1.30x1.75mm_HandSolder, F.Cu at (119.7, 132.9)
- added R11: 390, Resistor_SMD:R_1206_3216Metric_Pad1.30x1.75mm_HandSolder, F.Cu at (136.4, 131.8)
- added R12: 390, Resistor_SMD:R_1206_3216Metric_Pad1.30x1.75mm_HandSolder, F.Cu at (130.5, 131.8)
- added R13: 390, Resistor_SMD:R_1206_3216Metric_Pad1.30x1.75mm_HandSolder, F.Cu at (210.1, 82.1)
- added R14: 390, Resistor_SMD:R_1206_3216Metric_Pad1.30x1.75mm_HandSolder, F.Cu at (220.8, 81.0)
- added R15: 390, Resistor_SMD:R_1206_3216Metric_Pad1.30x1.75mm_HandSolder, F.Cu at (226.8, 81.0)
- added R16: 390, Resistor_SMD:R_1206_3216Metric_Pad1.30x1.75mm_HandSolder, F.Cu at (145.4, 132.9)
- added R17: 390, Resistor_SMD:R_1206_3216Metric_Pad1.30x1.75mm_HandSolder, F.Cu at (156.2, 131.8)
- added R18: 390, Resistor_SMD:R_1206_3216Metric_Pad1.30x1.75mm_HandSolder, F.Cu at (162.2, 131.8)
- added R19: 390, Resistor_SMD:R_1206_3216Metric_Pad1.30x1.75mm_HandSolder, F.Cu at (210.1, 97.9)
- added R2: 470 ohm, Resistor_SMD:R_1206_3216Metric_Pad1.30x1.75mm_HandSolder, F.Cu at (120.4, 63.0)
- added R20: 390, Resistor_SMD:R_1206_3216Metric_Pad1.30x1.75mm_HandSolder, F.Cu at (220.8, 96.8)
- added R21: 390, Resistor_SMD:R_1206_3216Metric_Pad1.30x1.75mm_HandSolder, F.Cu at (226.8, 96.8)
- added R22: 390, Resistor_SMD:R_1206_3216Metric_Pad1.30x1.75mm_HandSolder, F.Cu at (187.9, 131.8)
- added R23: 390, Resistor_SMD:R_1206_3216Metric_Pad1.30x1.75mm_HandSolder, F.Cu at (182.0, 131.8)
- added R24: 390, Resistor_SMD:R_1206_3216Metric_Pad1.30x1.75mm_HandSolder, F.Cu at (171.2, 132.9)
- added R25: 390, Resistor_SMD:R_1206_3216Metric_Pad1.30x1.75mm_HandSolder, F.Cu at (226.8, 112.6)
- added R26: 390, Resistor_SMD:R_1206_3216Metric_Pad1.30x1.75mm_HandSolder, F.Cu at (220.8, 112.6)
- added R27: 390, Resistor_SMD:R_1206_3216Metric_Pad1.30x1.75mm_HandSolder, F.Cu at (210.1, 113.7)
- added R3: 100 Kohm, Resistor_SMD:R_1206_3216Metric_Pad1.30x1.75mm_HandSolder, F.Cu at (120.4, 66.0)
- added R4: 390, Resistor_SMD:R_1206_3216Metric_Pad1.30x1.75mm_HandSolder, F.Cu at (94.0, 132.9)
- added R5: 390, Resistor_SMD:R_1206_3216Metric_Pad1.30x1.75mm_HandSolder, F.Cu at (104.7, 131.8)
- added R6: 390, Resistor_SMD:R_1206_3216Metric_Pad1.30x1.75mm_HandSolder, F.Cu at (110.7, 131.8)
- added R7: 390, Resistor_SMD:R_1206_3216Metric_Pad1.30x1.75mm_HandSolder, F.Cu at (210.1, 66.3)
- added R8: 390, Resistor_SMD:R_1206_3216Metric_Pad1.30x1.75mm_HandSolder, F.Cu at (220.8, 65.2)
- added R9: 390, Resistor_SMD:R_1206_3216Metric_Pad1.30x1.75mm_HandSolder, F.Cu at (226.8, 65.2)
- added U1: LM3671MF-3.3_NOPB, Package_TO_SOT_SMD:SOT-23, F.Cu at (114.6, 66.0)
- added U10: MOC3063, digikey-footprints:DIP-6_W7.62mm, F.Cu at (208.7, 104.9)
- added U2: PIC18F16Q40-E_SO, Package_SO:SOIC-20W_7.5x12.8mm_P1.27mm, F.Cu at (105.0, 67.9)
- added U3: MOC3063, digikey-footprints:DIP-6_W7.62mm, F.Cu at (92.5, 124.1)
- added U4: MOC3063, digikey-footprints:DIP-6_W7.62mm, F.Cu at (208.7, 57.5)
- added U5: MOC3063, digikey-footprints:DIP-6_W7.62mm, F.Cu at (118.3, 124.1)
- added U6: MOC3063, digikey-footprints:DIP-6_W7.62mm, F.Cu at (208.7, 73.3)
- added U7: MOC3063, digikey-footprints:DIP-6_W7.62mm, F.Cu at (144.1, 124.1)
- added U8: MOC3063, digikey-footprints:DIP-6_W7.62mm, F.Cu at (208.7, 89.1)
- added U9: MOC3063, digikey-footprints:DIP-6_W7.62mm, F.Cu at (169.8, 124.1)

Commit message: Before circuit change.
Parts:
- moved D1 84.7 mm to (161.3, 61.3)
- moved R4 84.7 mm to (148.6, 68.1)
- moved R5 84.7 mm to (159.3, 67.0)
- moved U3 84.7 mm to (147.2, 59.4)
- moved R6 84.7 mm to (165.3, 67.0)
- moved D3 59.7 mm to (161.6, 74.0)
- moved R10 59.7 mm to (148.9, 80.8)
- moved R11 59.7 mm to (165.6, 79.7)
- moved R12 59.7 mm to (159.7, 79.7)
- moved U5 59.7 mm to (147.5, 72.0)
- moved J2 55.8 mm to (109.2, 113.0)
- moved C1 53.4 mm to (119.4, 69.8)
- moved C4 47.3 mm to (119.4, 73.7)
- moved C3 45.3 mm to (126.0, 76.2), turned to 180 degrees
- moved D5 39.6 mm to (162.0, 86.7)
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
Commit message: Final attempt at single board.
Parts:
- removed C3: 22 uF, Capacitor_SMD:C_1206_3216Metric_Pad1.33x1.80mm_HandSolder
- removed C4: 0.1 uF 20V ceramic, Capacitor_SMD:C_1206_3216Metric_Pad1.33x1.80mm_HandSolder
- removed L1: 2.2 uH, Inductor_SMD:L_2816_7142Metric_Pad3.20x4.45mm_HandSolder
- removed R27: 390, Resistor_SMD:R_1206_3216Metric_Pad1.30x1.75mm_HandSolder
- removed U10: MOC3063, digikey-footprints:DIP-6_W7.62mm
- C1: value 10 uF -> 0.1 uF 20V ceramic; footprint Capacitor_SMD:C_1206_3216Metric_Pad1.33x1.80mm_HandSolder -> Capacitor_SMD:C_0805_2012Metric_Pad1.18x1.45mm_HandSolder
- C2: footprint Capacitor_SMD:C_1206_3216Metric_Pad1.33x1.80mm_HandSolder -> Capacitor_SMD:C_0805_2012Metric_Pad1.18x1.45mm_HandSolder
- J2: value GPIO Connector -> Input Connector; footprint Connector_PinHeader_2.54mm:PinHeader_1x05_P2.54mm_Vertical -> Connector_PinHeader_2.54mm:PinHeader_1x06_P2.54mm_Vertical
- J3: value Input Connector -> Output Connector
- J4: value Output Connector -> GPIO Connector; footprint Connector_PinHeader_2.54mm:PinHeader_1x06_P2.54mm_Vertical -> Connector_PinHeader_2.54mm:PinHeader_1x05_P2.54mm_Vertical
- R1, R10, R11, R12, R13, R14, R15, R16, R17, R18, R19, R2, R20, R21, R22, R23, R24, R25, R26, R4, R5, R6, R7, R8, R9: footprint Resistor_SMD:R_1206_3216Metric_Pad1.30x1.75mm_HandSolder -> Resistor_SMD:R_0805_2012Metric_Pad1.20x1.40mm_HandSolder
- R3: value 100 Kohm -> 390; footprint Resistor_SMD:R_1206_3216Metric_Pad1.30x1.75mm_HandSolder -> Resistor_SMD:R_0805_2012Metric_Pad1.20x1.40mm_HandSolder
- U1: value LM3671MF-3.3_NOPB -> PIC18F16Q40-E_SO; footprint Package_TO_SOT_SMD:SOT-23 -> Package_SO:SOIC-20W_7.5x12.8mm_P1.27mm
- U2: value PIC18F16Q40-E_SO -> MOC3063; footprint Package_SO:SOIC-20W_7.5x12.8mm_P1.27mm -> digikey-footprints:SMD-4_5x4.4mm_P4mm
- U3, U4, U5, U6, U7, U8, U9: footprint digikey-footprints:DIP-6_W7.62mm -> digikey-footprints:SMD-4_5x4.4mm_P4mm
- moved U2 66.3 mm to (158.6, 106.9)
- moved J1 59.7 mm to (110.5, 116.8)
- moved R3 54.2 mm to (146.6, 113.5)
- moved R9 50.2 mm to (152.0, 100.8)
- moved D1 48.1 mm to (149.2, 107.9)
- moved R5 47.1 mm to (151.4, 113.5)
- moved J2 45.8 mm to (134.6, 74.9), turned to 0 degrees
- moved R4 44.2 mm to (156.5, 111.6)
- moved R15 43.0 mm to (146.5, 88.1)
- moved R21 40.3 mm to (151.9, 75.4)
- moved U4 37.2 mm to (159.2, 94.2)
- moved R22 33.0 mm to (157.0, 73.5)
- moved R23 32.6 mm to (147.1, 75.4)
- moved D7 32.2 mm to (149.7, 69.8)
- moved U3 32.1 mm to (177.9, 68.5)
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Connections:
- C1 pad 1: +5V -> /Vpp
- C2 pad 1: /Vpp -> +3V3
- J1 pad 1: /ICSPCLK -> /Vpp
- J1 pad 2: /ICSPDAT -> +3V3
- J1 pad 4: +3V3 -> /ICSPDAT
- J1 pad 5: /Vpp -> /ICSPCLK
- J2 pad 1: /GPIO4 -> Net-(J2-Pad1)
- J2 pad 2: /GPIO3 -> HV_AC
- J2 pad 3: /GPIO2 -> /RX1
- J2 pad 4: /GPIO1 -> GND1
- J2 pad 5: /GPIO0 -> +3V3
- J3 pad 1: Net-(J3-Pad1) -> Net-(J2-Pad1)
- J3 pad 3: /RX1 -> /TX1
- J3 pad 5: +5V -> +3V3
- J4 pad 1: Net-(J3-Pad1) -> /GPIO4
- J4 pad 2: HV_AC -> /GPIO3
- J4 pad 3: /TX1 -> /GPIO2
- J4 pad 4: GND1 -> /GPIO1
- J4 pad 5: +5V -> /GPIO0
- R10 pad 1: Net-(R10-Pad1) -> HV_AC
- R10 pad 2: GND1 -> Net-(R10-Pad2)
- R11 pad 1: HV_AC -> /SegC
- R11 pad 2: Net-(R11-Pad2) -> Net-(D3-Pad3)
- R12 pad 1: /SegC -> Net-(R12-Pad1)
- R12 pad 2: Net-(D3-Pad3) -> GND1
- R13 pad 1: Net-(R13-Pad1) -> HV_AC
- R13 pad 2: GND1 -> Net-(R13-Pad2)
- R14 pad 1: HV_AC -> /SegD
- R14 pad 2: Net-(R14-Pad2) -> Net-(D4-Pad3)
- R15 pad 1: /SegD -> Net-(R15-Pad1)
- R15 pad 2: Net-(D4-Pad3) -> GND1
- R16 pad 1: Net-(R16-Pad1) -> HV_AC
- R16 pad 2: GND1 -> Net-(R16-Pad2)
- R17 pad 1: HV_AC -> /SegE
- R17 pad 2: Net-(R17-Pad2) -> Net-(D5-Pad3)
- R18 pad 1: /SegE -> Net-(R18-Pad1)
- R18 pad 2: Net-(D5-Pad3) -> GND1
- R19 pad 1: Net-(R19-Pad1) -> HV_AC
- R19 pad 2: GND1 -> Net-(R19-Pad2)
- R20 pad 1: HV_AC -> /SegF
- R20 pad 2: Net-(R20-Pad2) -> Net-(D6-Pad3)
- R21 pad 1: /SegF -> Net-(R21-Pad1)
- R21 pad 2: Net-(D6-Pad3) -> GND1
- R22 pad 1: Net-(R22-Pad1) -> HV_AC
- R22 pad 2: GND1 -> Net-(R22-Pad2)
- R23 pad 1: HV_AC -> /SegG
- R23 pad 2: Net-(R23-Pad2) -> Net-(D7-Pad3)
- R24 pad 1: /SegG -> Net-(R24-Pad1)
- R24 pad 2: Net-(D7-Pad3) -> GND1
- R25 pad 1: Net-(R25-Pad1) -> HV_AC
- R25 pad 2: GND1 -> Net-(R25-Pad2)
- R26 pad 1: HV_AC -> /SegH
- R26 pad 2: Net-(R26-Pad2) -> Net-(D8-Pad3)
- R3 pad 2: +5V -> GND1
- R4 pad 1: Net-(R4-Pad1) -> HV_AC
- R4 pad 2: GND1 -> Net-(R4-Pad2)
- R5 pad 1: HV_AC -> /SegA
- R5 pad 2: Net-(R5-Pad2) -> Net-(D1-Pad3)
- R6 pad 1: /SegA -> Net-(R6-Pad1)
- R6 pad 2: Net-(D1-Pad3) -> GND1
- R7 pad 1: Net-(R7-Pad1) -> HV_AC
- R7 pad 2: GND1 -> Net-(R7-Pad2)
- R8 pad 1: HV_AC -> /SegB
- R8 pad 2: Net-(R8-Pad2) -> Net-(D2-Pad3)
- R9 pad 1: /SegB -> Net-(R9-Pad1)
- R9 pad 2: Net-(D2-Pad3) -> GND1
- U1 pad 1: +5V -> +3V3
- U1 pad 2: GND -> /GPIO1
- U1 pad 3: Net-(R3-Pad1) -> /GPIO2
- U2 pad 1: +3V3 -> /EnbSegA
- U2 pad 2: /GPIO1 -> Net-(R3-Pad1)
- U2 pad 3: /GPIO2 -> Net-(U2-Pad3)
- U2 pad 4: /MCLR -> Net-(D1-Pad3)
- U3 pad 1: /EnbSegA -> /EnbSegB
- U3 pad 2: Net-(R4-Pad1) -> Net-(R6-Pad1)
- U3 pad 4: Net-(D1-Pad3) -> Net-(D2-Pad3)
- U4 pad 1: /EnbSegB -> /EnbSegC
- U4 pad 2: Net-(R7-Pad1) -> Net-(R9-Pad1)
- U4 pad 4: Net-(D2-Pad3) -> Net-(D3-Pad3)
- U5 pad 1: /EnbSegC -> /EnbSegD
- U5 pad 2: Net-(R10-Pad1) -> Net-(R12-Pad1)
- U5 pad 4: Net-(D3-Pad3) -> Net-(D4-Pad3)
- U6 pad 1: /EnbSegD -> /EnbSegE
- U6 pad 2: Net-(R13-Pad1) -> Net-(R15-Pad1)
- U6 pad 4: Net-(D4-Pad3) -> Net-(D5-Pad3)
- U7 pad 1: /EnbSegE -> /EnbSegF
- U7 pad 2: Net-(R16-Pad1) -> Net-(R18-Pad1)
- U7 pad 4: Net-(D5-Pad3) -> Net-(D6-Pad3)
- U8 pad 1: /EnbSegF -> /EnbSegG
- U8 pad 2: Net-(R19-Pad1) -> Net-(R21-Pad1)
- U8 pad 4: Net-(D6-Pad3) -> Net-(D7-Pad3)
- U9 pad 1: /EnbSegG -> /EnbSegH
- U9 pad 2: Net-(R22-Pad1) -> Net-(R24-Pad1)
- U9 pad 4: Net-(D7-Pad3) -> Net-(D8-Pad3)
