File: board/afdDriver/afdDriver.kicad_pcb (KiCad board)
At the start: 2 copper layers, 43.2 x 58.4 mm, 58 parts, among them J1 Qwiic_Connector, J2 Qwiic_Connector, J3 HighVoltageAC, J4 HighVoltageAC, J5 Power, U1 PCF8574TS, U2 QTM3063T1, U3 QTM3063T1, U4 QTM3063T1, U5 QTM3063T1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

Commit message: Fixed B.Mask text.
Other:
- board text added: "+5V"
- board text added: "GND"
Changed lines of the file:
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@@
   (general
     (thickness 1.6002)
-    (drawings 5)
+    (drawings 7)
     (tracks 648)
     (zones 0)
@@
       (effects (font (size 1 1) (thickness 0.15)) (justify mirror))
     )
-    (fp_text user 7 (at -19.05 -10.16) (layer B.SilkS)
+    (fp_text user 7 (at 18.8976 -10.6934) (layer B.SilkS)
       (effects (font (size 1 1) (thickness 0.15)) (justify mirror))
     )
-    (fp_text user 5 (at -19.05 -15.24) (layer B.SilkS)
+    (fp_text user 5 (at 18.7198 -15.24) (layer B.SilkS)
       (effects (font (size 1 1) (thickness 0.15)) (justify mirror))
     )
@@
     )
   )
+  (gr_text GND (at 106.8832 97.155) (layer B.SilkS)
+    (effects (font (size 1.524 1.524) (thickness 0.3048)) (justify mirror))
+  )
+  (gr_text +5V (at 101.8286 97.155) (layer B.SilkS)
+    (effects (font (size 1.524 1.524) (thickness 0.3048)) (justify mirror))
+  )
   (gr_text V1.0.0 (at 101.727 76.0476) (layer B.SilkS)

Commit message: Improved B.Silk layer on PCB. V1.0.1.
Other:
- board text added: "V1.0.1"
- board text removed: "V1.0.0"
Changed lines of the file:
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@@
   (title_block
     (title "Alien Font Display Driver Board")
-    (date 2021-12-07)
-    (rev V0.0.1)
+    (date 2021-12-12)
+    (rev V1.0.1)
     (comment 3 "MIT License")
   )
@@
     (effects (font (size 1.524 1.524) (thickness 0.3048)) (justify mirror))
   )
-  (gr_text V1.0.0 (at 101.727 76.0476) (layer B.SilkS)
+  (gr_text V1.0.1 (at 101.727 76.0476) (layer B.SilkS)
     (effects (font (size 0.8128 0.8128) (thickness 0.1524)) (justify mirror))
   )

Commit message: Improved RefDes for DS1 on B.Silk
Other:
- board text added: "V1.0.2"
- board text removed: "V1.0.1"
